Commit message: add castor joint to jointstate publisher

File: interncoxsys/urdf/model.urdf (robot description, URDF)
Before this commit: robot xxx, 24 links, 23 joints
Links:
- link base_link: geometry collision box size=0.65 0.55 0.25; visual mesh filename=file://src/interncoxsys/meshes/coconut.stl
